Commit message: 动态spawn: URDF自动同步Gazebo, 去掉home.world嵌死机器人

File: urdf/sensor_plugins.xacro (robot description, xacro)
@@ -1,5 +1,5 @@
 <?xml version="1.0"?>
 <robot name="sensor_plugins" xmlns:xacro="http://www.ros.org/wiki/xacro">
-<!-- Native Gazebo LiDAR on front_sensor_link -->
+<!-- GPU LiDAR on front_sensor_link -->
   <gazebo reference="front_sensor_link">
     <sensor name="front_lidar" type="gpu_lidar">
@@ -35,13 +35,6 @@
     </sensor>
   </gazebo>
-  <!-- Front camera optical frame (ROS convention: Z forward, X right, Y down) -->
-  <link name="front_camera_optical_frame"/>
-  <joint name="front_camera_optical_joint" type="fixed">
-    <parent link="front_sensor_link"/>
-    <child link="front_camera_optical_frame"/>
-    <origin xyz="0 0 0" rpy="-1.570796 0 -1.570796"/>
-  </joint>
-  <!-- Front camera sensor on front_sensor_link -->
-  <gazebo reference="front_sensor_link">
+  <!-- Camera sensor on rear_camera_link -->
+  <gazebo reference="rear_camera_link">
     <sensor name="front_camera" type="camera">
       <always_on>true</always_on>

Commit message: URDF加front_lidar link(RSP自动TF); 去掉被忽略的sensor内部pose

File: urdf/sensor_plugins.xacro (robot description, xacro)
@@ -4,5 +4,4 @@
   <gazebo reference="front_sensor_link">
     <sensor name="front_lidar" type="gpu_lidar">
-      <pose>0 0 0 0 1.570796 0</pose>
       <always_on>true</always_on>
       <update_rate>10</update_rate>

File: urdf/service_robot_cart_geometric.urdf.xacro (robot description, xacro)
@@ -873,3 +873,10 @@
     <origin xyz="-0.3525 0.0 0.11" rpy="0 0 3.141593"/>
   </joint>
+  <link name="front_lidar">
+  </link>
+  <joint name="front_lidar_joint" type="fixed">
+    <parent link="base_link"/>
+    <child link="front_lidar"/>
+    <origin xyz="0.0 0.0 0.20" rpy="0 0 3.141593"/>
+  </joint>
 </robot>

Commit message: 回退LiDAR配置: TF pitch=-90 yaw=180, 360度扫描, 无sensor内部pose

File: urdf/sensor_plugins.xacro (robot description, xacro)
@@ -1,5 +1,5 @@
 <?xml version="1.0"?>
 <robot name="sensor_plugins" xmlns:xacro="http://www.ros.org/wiki/xacro">
-<!-- GPU LiDAR on front_sensor_link. Internal pose counter-rotates scan to horizontal -->
+<!-- GPU LiDAR on front_sensor_link -->
   <gazebo reference="front_sensor_link">
     <sensor name="front_lidar" type="gpu_lidar">

File: urdf/service_robot_cart_geometric.urdf.xacro (robot description, xacro)
@@ -873,10 +873,3 @@
     <origin xyz="-0.3525 0.0 0.11" rpy="0 0 3.141593"/>
   </joint>
-  <link name="front_lidar">
-  </link>
-  <joint name="front_lidar_joint" type="fixed">
-    <parent link="base_link"/>
-    <child link="front_lidar"/>
-    <origin xyz="0.0 0.0 0.20" rpy="0 0 3.141593"/>
-  </joint>
 </robot>
