Commit message: home simulation: LiDAR夹层位 + TF/clock单调 + Nav2参数 + joint_states
- 激光雷达移至底座与第一货架夹层中间 (x=0, y=0, z=0.12)
- clock_bridge 加单调守卫, 拒绝 Gazebo 仿真时间回跳
- odom_bridge 改为使用 ROS wall time 而非 Gazebo 时间戳
- use_sim_time 全改为 false, 统一 wall time 避免 TF 时间跳变
- planner tolerance 0.5→2.0, robot_radius 0.4→0.25, costmap 30x30
- joint_vel_controller 发布 /joint_states 以支持 RSP 轮子 TF
- 新增 joint_state_publisher 节点消除 No transform 报错
- home.world: small_house SDF 1.9 + dartsim + JointControllerx4

File: urdf/service_robot_cart_geometric.urdf.xacro (robot description, xacro)
@@ -866,5 +866,5 @@
     <parent link="base_link"/>
     <child link="front_sensor_link"/>
-    <origin xyz="0.3025 0.0 0.11" rpy="0 0 0"/>
+    <origin xyz="0.0 0.0 0.12" rpy="0 0 0"/>
   </joint>
   <joint name="rear_sensor_link_joint" type="fixed">

Commit message: LiDAR: 上移3cm (z=0.12→0.15), 夹层中偏上

File: urdf/service_robot_cart_geometric.urdf.xacro (robot description, xacro)
@@ -866,5 +866,5 @@
     <parent link="base_link"/>
     <child link="front_sensor_link"/>
-    <origin xyz="0.0 0.0 0.12" rpy="0 0 0"/>
+    <origin xyz="0.0 0.0 0.15" rpy="0 0 0"/>
   </joint>
   <joint name="rear_sensor_link_joint" type="fixed">

Commit message: 货架上移6cm + LiDAR上移6cm(z=0.21) + roll 90deg

File: urdf/service_robot_cart_geometric.urdf.xacro (robot description, xacro)
@@ -758,5 +758,5 @@
     <parent link="base_link"/>
     <child link="body_link"/>
-    <origin xyz="-0.175 0.0 0.49" rpy="0 0 0"/>
+    <origin xyz="-0.175 0.0 0.55" rpy="0 0 0"/>
   </joint>
   <joint name="tray_1_joint" type="fixed">
@@ -866,5 +866,5 @@
     <parent link="base_link"/>
     <child link="front_sensor_link"/>
-    <origin xyz="0.0 0.0 0.15" rpy="0 0 0"/>
+    <origin xyz="0.0 0.0 0.21" rpy="1.570796 0 0"/>
   </joint>
   <joint name="rear_sensor_link_joint" type="fixed">

Commit message: fix: 只移tray(+6cm), 回退body_link; LiDAR z=0.21 roll=90deg

File: urdf/service_robot_cart_geometric.urdf.xacro (robot description, xacro)
@@ -758,10 +758,10 @@
     <parent link="base_link"/>
     <child link="body_link"/>
-    <origin xyz="-0.175 0.0 0.55" rpy="0 0 0"/>
+    <origin xyz="-0.175 0.0 0.49" rpy="0 0 0"/>
   </joint>
   <joint name="tray_1_joint" type="fixed">
     <parent link="body_link"/>
     <child link="tray_1_link"/>
-    <origin xyz="0.295 0.0 -0.275" rpy="0 0 0"/>
+    <origin xyz="0.295 0.0 -0.215" rpy="0 0 0"/>
   </joint>
   <joint name="tray_1_surface_frame_joint" type="fixed">
@@ -773,5 +773,5 @@
     <parent link="body_link"/>
     <child link="tray_2_link"/>
-    <origin xyz="0.295 0.0 -0.125" rpy="0 0 0"/>
+    <origin xyz="0.295 0.0 -0.065" rpy="0 0 0"/>
   </joint>
   <joint name="tray_2_surface_frame_joint" type="fixed">
@@ -783,5 +783,5 @@
     <parent link="body_link"/>
     <child link="tray_3_link"/>
-    <origin xyz="0.295 0.0 0.025" rpy="0 0 0"/>
+    <origin xyz="0.295 0.0 0.085" rpy="0 0 0"/>
   </joint>
   <joint name="tray_3_surface_frame_joint" type="fixed">
@@ -793,5 +793,5 @@
     <parent link="body_link"/>
     <child link="tray_4_link"/>
-    <origin xyz="0.295 0.0 0.175" rpy="0 0 0"/>
+    <origin xyz="0.295 0.0 0.235" rpy="0 0 0"/>
   </joint>
   <joint name="tray_4_surface_frame_joint" type="fixed">

Commit message: LiDAR: roll→pitch 90deg (Y轴旋转, 前后垂直扫描)

File: urdf/service_robot_cart_geometric.urdf.xacro (robot description, xacro)
@@ -866,5 +866,5 @@
     <parent link="base_link"/>
     <child link="front_sensor_link"/>
-    <origin xyz="0.0 0.0 0.21" rpy="1.570796 0 0"/>
+    <origin xyz="0.0 0.0 0.21" rpy="0 1.570796 0"/>
   </joint>
   <joint name="rear_sensor_link_joint" type="fixed">

Commit message: LiDAR 顺时针180deg + 下移3cm(z=0.18); 货架整体-3cm

File: urdf/service_robot_cart_geometric.urdf.xacro (robot description, xacro)
@@ -552,5 +552,5 @@
     </visual>
     <visual name="rear_camera_silver_ring">
-      <origin xyz="0.0125 0.0 0.0225" rpy="0 1.570796 0"/>
+      <origin xyz="0.0125 0.0 0.0225" rpy="0 1.570796 3.141593"/>
       <geometry>
         <cylinder radius="0.035" length="0.02"/>
@@ -559,5 +559,5 @@
     </visual>
     <visual name="rear_camera_glass_lens">
-      <origin xyz="0.025 0.0 0.0225" rpy="0 1.570796 0"/>
+      <origin xyz="0.025 0.0 0.0225" rpy="0 1.570796 3.141593"/>
       <geometry>
         <cylinder radius="0.0225" length="0.022"/>
@@ -595,5 +595,5 @@
     </inertial>
     <visual name="left_side_camera_housing">
-      <origin xyz="0.0 0.0 0.0" rpy="0 1.570796 0"/>
+      <origin xyz="0.0 0.0 0.0" rpy="0 1.570796 3.141593"/>
       <geometry>
         <cylinder radius="0.0325" length="0.0275"/>
@@ -602,5 +602,5 @@
     </visual>
     <visual name="left_side_camera_lens">
-      <origin xyz="0.013 0.0 0.0" rpy="0 1.570796 0"/>
+      <origin xyz="0.013 0.0 0.0" rpy="0 1.570796 3.141593"/>
       <geometry>
         <cylinder radius="0.02" length="0.03"/>
@@ -609,5 +609,5 @@
     </visual>
     <visual name="left_side_camera_black_ring">
-      <origin xyz="0.01 0.0 0.0" rpy="0 1.570796 0"/>
+      <origin xyz="0.01 0.0 0.0" rpy="0 1.570796 3.141593"/>
       <geometry>
         <cylinder radius="0.0235" length="0.032"/>
@@ -616,5 +616,5 @@
     </visual>
     <collision name="left_side_camera_link_collision">
-      <origin xyz="0.0 0.0 0.0" rpy="0 1.570796 0"/>
+      <origin xyz="0.0 0.0 0.0" rpy="0 1.570796 3.141593"/>
       <geometry>
         <cylinder radius="0.035" length="0.035"/>
@@ -631,5 +631,5 @@
     </inertial>
     <visual name="right_side_camera_housing">
-      <origin xyz="0.0 0.0 0.0" rpy="0 1.570796 0"/>
+      <origin xyz="0.0 0.0 0.0" rpy="0 1.570796 3.141593"/>
       <geometry>
         <cylinder radius="0.0325" length="0.0275"/>
@@ -638,5 +638,5 @@
     </visual>
     <visual name="right_side_camera_lens">
-      <origin xyz="0.013 0.0 0.0" rpy="0 1.570796 0"/>
+      <origin xyz="0.013 0.0 0.0" rpy="0 1.570796 3.141593"/>
       <geometry>
         <cylinder radius="0.02" length="0.03"/>
@@ -645,5 +645,5 @@
     </visual>
     <visual name="right_side_camera_black_ring">
-      <origin xyz="0.01 0.0 0.0" rpy="0 1.570796 0"/>
+      <origin xyz="0.01 0.0 0.0" rpy="0 1.570796 3.141593"/>
       <geometry>
         <cylinder radius="0.0235" length="0.032"/>
@@ -652,5 +652,5 @@
     </visual>
     <collision name="right_side_camera_link_collision">
-      <origin xyz="0.0 0.0 0.0" rpy="0 1.570796 0"/>
+      <origin xyz="0.0 0.0 0.0" rpy="0 1.570796 3.141593"/>
       <geometry>
         <cylinder radius="0.035" length="0.035"/>
@@ -708,5 +708,5 @@
     </inertial>
     <visual name="front_sensor_link_silver_ring">
-      <origin xyz="0.0 0.0 0.0" rpy="0 1.570796 0"/>
+      <origin xyz="0.0 0.0 0.0" rpy="0 1.570796 3.141593"/>
       <geometry>
         <cylinder radius="0.02" length="0.0125"/>
@@ -715,5 +715,5 @@
     </visual>
     <visual name="front_sensor_link_glass">
-      <origin xyz="0.006 0.0 0.0" rpy="0 1.570796 0"/>
+      <origin xyz="0.006 0.0 0.0" rpy="0 1.570796 3.141593"/>
       <geometry>
         <cylinder radius="0.013" length="0.015"/>
@@ -722,5 +722,5 @@
     </visual>
     <collision name="front_sensor_link_collision">
-      <origin xyz="0.0 0.0 0.0" rpy="0 1.570796 0"/>
+      <origin xyz="0.0 0.0 0.0" rpy="0 1.570796 3.141593"/>
       <geometry>
         <cylinder radius="0.0225" length="0.0175"/>
@@ -735,5 +735,5 @@
     </inertial>
     <visual name="rear_sensor_link_silver_ring">
-      <origin xyz="0.0 0.0 0.0" rpy="0 1.570796 0"/>
+      <origin xyz="0.0 0.0 0.0" rpy="0 1.570796 3.141593"/>
       <geometry>
         <cylinder radius="0.02" length="0.0125"/>
@@ -742,5 +742,5 @@
     </visual>
     <visual name="rear_sensor_link_glass">
-      <origin xyz="0.006 0.0 0.0" rpy="0 1.570796 0"/>
+      <origin xyz="0.006 0.0 0.0" rpy="0 1.570796 3.141593"/>
       <geometry>
         <cylinder radius="0.013" length="0.015"/>
@@ -749,5 +749,5 @@
     </visual>
     <collision name="rear_sensor_link_collision">
-      <origin xyz="0.0 0.0 0.0" rpy="0 1.570796 0"/>
+      <origin xyz="0.0 0.0 0.0" rpy="0 1.570796 3.141593"/>
       <geometry>
         <cylinder radius="0.0225" length="0.0175"/>
@@ -763,5 +763,5 @@
     <parent link="body_link"/>
     <child link="tray_1_link"/>
-    <origin xyz="0.295 0.0 -0.215" rpy="0 0 0"/>
+    <origin xyz="0.295 0.0 -0.245" rpy="0 0 0"/>
   </joint>
   <joint name="tray_1_surface_frame_joint" type="fixed">
@@ -773,5 +773,5 @@
     <parent link="body_link"/>
     <child link="tray_2_link"/>
-    <origin xyz="0.295 0.0 -0.065" rpy="0 0 0"/>
+    <origin xyz="0.295 0.0 -0.095" rpy="0 0 0"/>
   </joint>
   <joint name="tray_2_surface_frame_joint" type="fixed">
@@ -783,5 +783,5 @@
     <parent link="body_link"/>
     <child link="tray_3_link"/>
-    <origin xyz="0.295 0.0 0.085" rpy="0 0 0"/>
+    <origin xyz="0.295 0.0 0.055" rpy="0 0 0"/>
   </joint>
   <joint name="tray_3_surface_frame_joint" type="fixed">
@@ -793,5 +793,5 @@
     <parent link="body_link"/>
     <child link="tray_4_link"/>
-    <origin xyz="0.295 0.0 0.235" rpy="0 0 0"/>
+    <origin xyz="0.295 0.0 0.205" rpy="0 0 0"/>
   </joint>
   <joint name="tray_4_surface_frame_joint" type="fixed">
@@ -866,5 +866,5 @@
     <parent link="base_link"/>
     <child link="front_sensor_link"/>
-    <origin xyz="0.0 0.0 0.21" rpy="0 1.570796 0"/>
+    <origin xyz="0.0 0.0 0.18" rpy="0 1.570796 3.141593"/>
   </joint>
   <joint name="rear_sensor_link_joint" type="fixed">

Commit message: LiDAR 上移2cm (z=0.18→0.20)

File: urdf/service_robot_cart_geometric.urdf.xacro (robot description, xacro)
@@ -866,5 +866,5 @@
     <parent link="base_link"/>
     <child link="front_sensor_link"/>
-    <origin xyz="0.0 0.0 0.18" rpy="0 1.570796 3.141593"/>
+    <origin xyz="0.0 0.0 0.20" rpy="0 1.570796 3.141593"/>
   </joint>
   <joint name="rear_sensor_link_joint" type="fixed">

Commit message: LiDAR pitch +180deg→-90deg; 扫描360→180(背向body_link半面屏蔽)

File: urdf/service_robot_cart_geometric.urdf.xacro (robot description, xacro)
@@ -552,5 +552,5 @@
     </visual>
     <visual name="rear_camera_silver_ring">
-      <origin xyz="0.0125 0.0 0.0225" rpy="0 1.570796 3.141593"/>
+      <origin xyz="0.0125 0.0 0.0225" rpy="0 -1.570796 3.141593"/>
       <geometry>
         <cylinder radius="0.035" length="0.02"/>
@@ -559,5 +559,5 @@
     </visual>
     <visual name="rear_camera_glass_lens">
-      <origin xyz="0.025 0.0 0.0225" rpy="0 1.570796 3.141593"/>
+      <origin xyz="0.025 0.0 0.0225" rpy="0 -1.570796 3.141593"/>
       <geometry>
         <cylinder radius="0.0225" length="0.022"/>
@@ -595,5 +595,5 @@
     </inertial>
     <visual name="left_side_camera_housing">
-      <origin xyz="0.0 0.0 0.0" rpy="0 1.570796 3.141593"/>
+      <origin xyz="0.0 0.0 0.0" rpy="0 -1.570796 3.141593"/>
       <geometry>
         <cylinder radius="0.0325" length="0.0275"/>
@@ -602,5 +602,5 @@
     </visual>
     <visual name="left_side_camera_lens">
-      <origin xyz="0.013 0.0 0.0" rpy="0 1.570796 3.141593"/>
+      <origin xyz="0.013 0.0 0.0" rpy="0 -1.570796 3.141593"/>
       <geometry>
         <cylinder radius="0.02" length="0.03"/>
@@ -609,5 +609,5 @@
     </visual>
     <visual name="left_side_camera_black_ring">
-      <origin xyz="0.01 0.0 0.0" rpy="0 1.570796 3.141593"/>
+      <origin xyz="0.01 0.0 0.0" rpy="0 -1.570796 3.141593"/>
       <geometry>
         <cylinder radius="0.0235" length="0.032"/>
@@ -616,5 +616,5 @@
     </visual>
     <collision name="left_side_camera_link_collision">
-      <origin xyz="0.0 0.0 0.0" rpy="0 1.570796 3.141593"/>
+      <origin xyz="0.0 0.0 0.0" rpy="0 -1.570796 3.141593"/>
       <geometry>
         <cylinder radius="0.035" length="0.035"/>
@@ -631,5 +631,5 @@
     </inertial>
     <visual name="right_side_camera_housing">
-      <origin xyz="0.0 0.0 0.0" rpy="0 1.570796 3.141593"/>
+      <origin xyz="0.0 0.0 0.0" rpy="0 -1.570796 3.141593"/>
       <geometry>
         <cylinder radius="0.0325" length="0.0275"/>
@@ -638,5 +638,5 @@
     </visual>
     <visual name="right_side_camera_lens">
-      <origin xyz="0.013 0.0 0.0" rpy="0 1.570796 3.141593"/>
+      <origin xyz="0.013 0.0 0.0" rpy="0 -1.570796 3.141593"/>
       <geometry>
         <cylinder radius="0.02" length="0.03"/>
@@ -645,5 +645,5 @@
     </visual>
     <visual name="right_side_camera_black_ring">
-      <origin xyz="0.01 0.0 0.0" rpy="0 1.570796 3.141593"/>
+      <origin xyz="0.01 0.0 0.0" rpy="0 -1.570796 3.141593"/>
       <geometry>
         <cylinder radius="0.0235" length="0.032"/>
@@ -652,5 +652,5 @@
     </visual>
     <collision name="right_side_camera_link_collision">
-      <origin xyz="0.0 0.0 0.0" rpy="0 1.570796 3.141593"/>
+      <origin xyz="0.0 0.0 0.0" rpy="0 -1.570796 3.141593"/>
       <geometry>
         <cylinder radius="0.035" length="0.035"/>
@@ -708,5 +708,5 @@
     </inertial>
     <visual name="front_sensor_link_silver_ring">
-      <origin xyz="0.0 0.0 0.0" rpy="0 1.570796 3.141593"/>
+      <origin xyz="0.0 0.0 0.0" rpy="0 -1.570796 3.141593"/>
       <geometry>
         <cylinder radius="0.02" length="0.0125"/>
@@ -715,5 +715,5 @@
     </visual>
     <visual name="front_sensor_link_glass">
-      <origin xyz="0.006 0.0 0.0" rpy="0 1.570796 3.141593"/>
+      <origin xyz="0.006 0.0 0.0" rpy="0 -1.570796 3.141593"/>
       <geometry>
         <cylinder radius="0.013" length="0.015"/>
@@ -722,5 +722,5 @@
     </visual>
     <collision name="front_sensor_link_collision">
-      <origin xyz="0.0 0.0 0.0" rpy="0 1.570796 3.141593"/>
+      <origin xyz="0.0 0.0 0.0" rpy="0 -1.570796 3.141593"/>
       <geometry>
         <cylinder radius="0.0225" length="0.0175"/>
@@ -735,5 +735,5 @@
     </inertial>
     <visual name="rear_sensor_link_silver_ring">
-      <origin xyz="0.0 0.0 0.0" rpy="0 1.570796 3.141593"/>
+      <origin xyz="0.0 0.0 0.0" rpy="0 -1.570796 3.141593"/>
       <geometry>
         <cylinder radius="0.02" length="0.0125"/>
@@ -742,5 +742,5 @@
     </visual>
     <visual name="rear_sensor_link_glass">
-      <origin xyz="0.006 0.0 0.0" rpy="0 1.570796 3.141593"/>
+      <origin xyz="0.006 0.0 0.0" rpy="0 -1.570796 3.141593"/>
       <geometry>
         <cylinder radius="0.013" length="0.015"/>
@@ -749,5 +749,5 @@
     </visual>
     <collision name="rear_sensor_link_collision">
-      <origin xyz="0.0 0.0 0.0" rpy="0 1.570796 3.141593"/>
+      <origin xyz="0.0 0.0 0.0" rpy="0 -1.570796 3.141593"/>
       <geometry>
         <cylinder radius="0.0225" length="0.0175"/>
@@ -866,5 +866,5 @@
     <parent link="base_link"/>
     <child link="front_sensor_link"/>
-    <origin xyz="0.0 0.0 0.20" rpy="0 1.570796 3.141593"/>
+    <origin xyz="0.0 0.0 0.20" rpy="0 -1.570796 3.141593"/>
   </joint>
   <joint name="rear_sensor_link_joint" type="fixed">

Commit message: tray整体上移3cm (URDF+SDF同步)

File: urdf/service_robot_cart_geometric.urdf.xacro (robot description, xacro)
@@ -763,5 +763,5 @@
     <parent link="body_link"/>
     <child link="tray_1_link"/>
-    <origin xyz="0.295 0.0 -0.245" rpy="0 0 0"/>
+    <origin xyz="0.295 0.0 -0.215" rpy="0 0 0"/>
   </joint>
   <joint name="tray_1_surface_frame_joint" type="fixed">
@@ -773,5 +773,5 @@
     <parent link="body_link"/>
     <child link="tray_2_link"/>
-    <origin xyz="0.295 0.0 -0.095" rpy="0 0 0"/>
+    <origin xyz="0.295 0.0 -0.065" rpy="0 0 0"/>
   </joint>
   <joint name="tray_2_surface_frame_joint" type="fixed">
@@ -783,5 +783,5 @@
     <parent link="body_link"/>
     <child link="tray_3_link"/>
-    <origin xyz="0.295 0.0 0.055" rpy="0 0 0"/>
+    <origin xyz="0.295 0.0 0.085" rpy="0 0 0"/>
   </joint>
   <joint name="tray_3_surface_frame_joint" type="fixed">
@@ -793,5 +793,5 @@
     <parent link="body_link"/>
     <child link="tray_4_link"/>
-    <origin xyz="0.295 0.0 0.205" rpy="0 0 0"/>
+    <origin xyz="0.295 0.0 0.235" rpy="0 0 0"/>
   </joint>
   <joint name="tray_4_surface_frame_joint" type="fixed">
